Commit message: fix joint name; incorrectly referenced panda_hand_joint

File: armada_description/urdf/modules/mounts/mpm/mount.xacro (robot description, xacro)
@@ -6,5 +6,5 @@
 <!-- =================================================================================== -->
     <xacro:macro name="armada_mount" params="prefix parent *origin" >
-        <joint name="panda_hand_joint" type="fixed">
+        <joint name="flange_mpm_joint" type="fixed">
             <parent link="${parent}" />
             <child link="${prefix}base_link" />
@@ -14,10 +14,10 @@
             <visual>
                 <geometry>
-                    <mesh filename="file://$(find armada_description)/meshes/modules/mpm/visual/mpm.stl" />
+                    <mesh filename="file://$(find armada_description)/meshes/modules/mounts/mpm/visual/mpm.stl" />
                 </geometry>
             </visual>
             <collision>
                 <geometry>
-                    <mesh filename="file://$(find armada_description)/meshes/modules/mpm/collision/mpm.stl" />
+                    <mesh filename="file://$(find armada_description)/meshes/modules//mounts/mpm/collision/mpm.stl" />
                 </geometry>
             </collision>
