Commit message: remove name and tf_prefix args, pass tf_prefix to macro directly and use value for tf_prefix param in subsequent ur_robot macro

File: armada_description/urdf/modules/arms/ur5e/arm.xacro (robot description, xacro)
@@ -4,7 +4,4 @@
   <xacro:include filename="$(find ur_description)/urdf/ur_macro.xacro"/>
   <!-- UR5e-specific defaults -->
-  <xacro:arg name="name" default="ur5e"/>
-  <!-- <xacro:arg name="tf_prefix" default="ur5e_"/> -->
-  <xacro:arg name="tf_prefix" default=""/>
   <xacro:arg name="joint_limit_params"
               default="$(find ur_description)/config/ur5e/joint_limits.yaml"/>
@@ -19,8 +16,8 @@
   <xacro:arg name="safety_k_position" default="20"/>
   <!-- Generic macro expected by robot.urdf.xacro -->
-  <xacro:macro name="armada_arm" params="parent *origin">
+  <xacro:macro name="armada_arm" params="tf_prefix parent *origin">
     <xacro:ur_robot
-      name="$(arg name)"
-      tf_prefix="$(arg tf_prefix)"
+      name=""
+      tf_prefix="${tf_prefix}"
       parent="${parent}"
       joint_limits_parameters_file="$(arg joint_limit_params)"
