Commit message: tcp_link added to robot to allow kinematic chain extension to plan about tcp, will need to be moved later or adjusted to be more easily modifiable/parameterized

File: armada_description/urdf/modules/arms/ur5e/arm.xacro (robot description, xacro)
@@ -28,4 +28,11 @@
       <xacro:insert_block name="origin"/>
     </xacro:ur_robot>
+    <!-- Prototype manipulation TCP, 21 cm along the tool0 +Z axis. -->
+    <link name="tcp_link"/>
+    <joint name="${tf_prefix}tool0_tcp_joint" type="fixed">
+      <parent link="${tf_prefix}tool0"/>
+      <child link="tcp_link"/>
+      <origin xyz="0 0 0.21" rpy="0 0 0"/>
+    </joint>
   </xacro:macro>
 </robot>

Commit message: modify tcp_link length, too far from actual grasping point

File: armada_description/urdf/modules/arms/ur5e/arm.xacro (robot description, xacro)
@@ -33,5 +33,5 @@
       <parent link="${tf_prefix}tool0"/>
       <child link="tcp_link"/>
-      <origin xyz="0 0 0.21" rpy="0 0 0"/>
+      <origin xyz="0 0 0.195" rpy="0 0 0"/>
     </joint>
   </xacro:macro>

Commit message: increase tcp distance after further testing

File: armada_description/urdf/modules/arms/ur5e/arm.xacro (robot description, xacro)
@@ -33,5 +33,5 @@
       <parent link="${tf_prefix}tool0"/>
       <child link="tcp_link"/>
-      <origin xyz="0 0 0.195" rpy="0 0 0"/>
+      <origin xyz="0 0 0.21" rpy="0 0 0"/>
     </joint>
   </xacro:macro>
