Commit message: load ur.ros2_control.xacro macro for actual hardware, passing through required default values

File: armada_description/urdf/modules/arms/ur5e/ros2_control.xacro (robot description, xacro)
@@ -1,19 +1,62 @@
 <?xml version="1.0"?>
 <robot xmlns:xacro="http://www.ros.org/wiki/xacro">
-  <xacro:include filename="$(find ur_description)/urdf/inc/ur_joint_control.xacro" />
-  <xacro:macro name="armada_arm_ros2_control" params="
-      prefix
-      initial_positions:=${dict(shoulder_pan_joint=0.0,shoulder_lift_joint=-1.57,elbow_joint=0.0,wrist_1_joint=-1.57,wrist_2_joint=0.0,wrist_3_joint=0.0)}
-    ">
-    <ros2_control name="${prefix}ur_arm_ros2_control" type="system">
-      <hardware>
-        <!-- Gazebo Sim -->
-        <plugin>gz_ros2_control/GazeboSimSystem</plugin>
-      </hardware>
-      <xacro:ur_joint_control_description
-        tf_prefix="${prefix}"
-        initial_positions="${initial_positions}"
-      />
-    </ros2_control>
+  <!-- Load the real UR ros2_control macro -->
+  <xacro:include filename="$(find ur_robot_driver)/urdf/ur.ros2_control.xacro"/>
+  <!-- UR5e-specific constants/defaults -->
+  <xacro:arg name="robot_ip" default="0.0.0.0"/>
+  <xacro:arg name="reverse_ip" default="0.0.0.0"/>
+  <xacro:arg name="use_mock_hardware" default="false"/>
+  <xacro:arg name="mock_sensor_commands" default="false"/>
+  <xacro:arg name="headless_mode" default="false"/>
+  <xacro:arg name="script_filename" default=""/>
+  <xacro:arg name="output_recipe_filename" default=""/>
+  <xacro:arg name="input_recipe_filename" default=""/>
+  <xacro:arg name="script_command_port" default="50004"/>
+  <xacro:arg name="reverse_port" default="50001"/>
+  <xacro:arg name="script_sender_port" default="50002"/>
+  <xacro:arg name="trajectory_port" default="50003"/>
+  <xacro:arg name="use_tool_communication" default="false"/>
+  <xacro:arg name="tool_voltage" default="0"/>
+  <xacro:arg name="tool_parity" default="0"/>
+  <xacro:arg name="tool_baud_rate" default="115200"/>
+  <xacro:arg name="tool_stop_bits" default="1"/>
+  <xacro:arg name="tool_rx_idle_chars" default="1.5"/>
+  <xacro:arg name="tool_tx_idle_chars" default="3.5"/>
+  <xacro:arg name="tool_device_name" default="/tmp/ttyUR"/>
+  <xacro:arg name="tool_tcp_port" default="54321"/>
+  <xacro:arg name="initial_positions_file"
+              default="$(find ur_description)/config/initial_positions.yaml"/>
+  <xacro:property name="initial_positions_file"
+                  value="$(arg initial_positions_file)"/>
+  <!-- This is the generic macro your robot.urdf.xacro calls -->
+  <xacro:macro name="armada_arm_ros2_control" params="prefix">
+    <xacro:ur_ros2_control
+      name="${prefix}ur_system"
+      tf_prefix="${prefix}"
+      kinematics_parameters_file="$(find ur_description)/config/ur5e/default_kinematics.yaml"
+      transmission_hw_interface="hardware_interface/PositionJointInterface"
+      use_mock_hardware="$(arg use_mock_hardware)"
+      mock_sensor_commands="$(arg mock_sensor_commands)"
+      headless_mode="$(arg headless_mode)"
+      initial_positions="${xacro.load_yaml(initial_positions_file)}"
+      use_tool_communication="$(arg use_tool_communication)"
+      tool_voltage="$(arg tool_voltage)"
+      tool_parity="$(arg tool_parity)"
+      tool_baud_rate="$(arg tool_baud_rate)"
+      tool_stop_bits="$(arg tool_stop_bits)"
+      tool_rx_idle_chars="$(arg tool_rx_idle_chars)"
+      tool_tx_idle_chars="$(arg tool_tx_idle_chars)"
+      tool_device_name="$(arg tool_device_name)"
+      tool_tcp_port="$(arg tool_tcp_port)"
+      robot_ip="$(arg robot_ip)"
+      script_filename="$(arg script_filename)"
+      output_recipe_filename="$(arg output_recipe_filename)"
+      input_recipe_filename="$(arg input_recipe_filename)"
+      reverse_ip="$(arg reverse_ip)"
+      script_command_port="$(arg script_command_port)"
+      reverse_port="$(arg reverse_port)"
+      script_sender_port="$(arg script_sender_port)"
+      trajectory_port="$(arg trajectory_port)"
+    />
   </xacro:macro>
 </robot>

Commit message: add ur_ros2_control macro call from ur_description package, pass through robot_ip and prefix args

File: armada_description/urdf/modules/arms/ur5e/ros2_control.xacro (robot description, xacro)
@@ -30,5 +30,5 @@
                   value="$(arg initial_positions_file)"/>
   <!-- This is the generic macro your robot.urdf.xacro calls -->
-  <xacro:macro name="armada_arm_ros2_control" params="prefix">
+  <xacro:macro name="armada_arm_ros2_control" params="prefix robot_ip">
     <xacro:ur_ros2_control
       name="${prefix}ur_system"

Commit message: add ur_type param back, apply model to ur_type to maintain structure

File: armada_description/urdf/modules/arms/ur5e/ros2_control.xacro (robot description, xacro)
@@ -30,8 +30,9 @@
                   value="$(arg initial_positions_file)"/>
   <!-- This is the generic macro your robot.urdf.xacro calls -->
-  <xacro:macro name="armada_arm_ros2_control" params="prefix robot_ip">
+  <xacro:macro name="armada_arm_ros2_control" params="prefix robot_ip model">
     <xacro:ur_ros2_control
       name="${prefix}ur_system"
       tf_prefix="${prefix}"
+      ur_type="${model}"
       kinematics_parameters_file="$(find ur_description)/config/ur5e/default_kinematics.yaml"
       transmission_hw_interface="hardware_interface/PositionJointInterface"

Commit message: point to actual extracted robot config file as per ur instructions, make some formatting adjustments for visual clarity

File: armada_description/urdf/modules/arms/ur5e/ros2_control.xacro (robot description, xacro)
@@ -25,8 +25,6 @@
   <xacro:arg name="tool_device_name" default="/tmp/ttyUR"/>
   <xacro:arg name="tool_tcp_port" default="54321"/>
-  <xacro:arg name="initial_positions_file"
-              default="$(find ur_description)/config/initial_positions.yaml"/>
-  <xacro:property name="initial_positions_file"
-                  value="$(arg initial_positions_file)"/>
+  <xacro:arg name="initial_positions_file" default="$(find ur_description)/config/initial_positions.yaml"/>
+  <xacro:property name="initial_positions_file" value="$(arg initial_positions_file)"/>
   <!-- This is the generic macro your robot.urdf.xacro calls -->
   <xacro:macro name="armada_arm_ros2_control" params="prefix robot_ip model">
@@ -35,5 +33,5 @@
       tf_prefix="${prefix}"
       ur_type="${model}"
-      kinematics_parameters_file="$(find ur_description)/config/ur5e/default_kinematics.yaml"
+      kinematics_parameters_file="$(find armada_bringup)/config/modules/arms/ur5e/ur5e_calibration.yaml"
       transmission_hw_interface="hardware_interface/PositionJointInterface"
       use_mock_hardware="$(arg use_mock_hardware)"
