Commit message: replace cylinder geometry with ur_to_robotiq_adapter model files and use inertiavalues from same robotiq package

File: armada_description/urdf/modules/end_effectors/robotiq_2f85/cable_adapter.xacro (robot description, xacro)
@@ -1,8 +1,4 @@
 <?xml version="1.0" ?>
 <robot xmlns:xacro="http://www.ros.org/wiki/xacro" name="r2f85_connector_adapter_description">
-<!-- =================================================================================== -->
-<!-- |    This document was autogenerated by xacro from /opt/ros/kinetic/share/moveit_resources/panda_description/urdf/panda.urdf | -->
-<!-- |    EDITING THIS FILE BY HAND IS NOT RECOMMENDED                                 | -->
-<!-- =================================================================================== -->
     <xacro:macro name="armada_ee_connector_adapter" params="prefix parent *origin" >
         <joint name="flange_ee_connector_adapter_joint" type="fixed">
@@ -14,20 +10,17 @@
             <visual>
                 <geometry>
-                    <cylinder radius="0.0375" length="0.017"/>
+                    <mesh filename="package://robotiq_description/meshes/visual/2f_85/ur_to_robotiq_adapter.dae"/>
                 </geometry>
             </visual>
             <collision>
                 <geometry>
-                    <cylinder radius="0.0375" length="0.017"/>
+                    <mesh filename="package://robotiq_description/meshes/collision/2f_85/ur_to_robotiq_adapter.stl"/>
                 </geometry>
             </collision>
             <inertial>
-            <origin xyz="0 0 0" rpy="0 0 0" />
-            <mass value="0.01"/>
-            <inertia
-                ixx="1e-5" ixy="0" ixz="0"
-                iyy="1e-5" iyz="0"
-                izz="1e-5"/>
-            </inertial>
+                <origin xyz="0 0 0" rpy="0 0 0" />
+                <mass value="0.01"/>
+                <inertia ixx="0.000044" ixy="0.0" ixz="0.0" iyy="0.000027" iyz="0.0" izz="0.000027" />
+            </inertial> -->
         </link>
     </xacro:macro>
