Commit message: add material and color tag to visual geometry so model doesn't appear red; can be misinterpreted as a detected collision

File: armada_description/urdf/modules/controllers/rpi5_enclosure/controller.xacro (robot description, xacro)
@@ -16,4 +16,7 @@
                     <box size="0.065 0.095 0.035"/>
                 </geometry>
+                <material name="gray">
+                    <color rgba="0.7 0.7 0.7 1.0"/>
+                </material>
             </visual>
             <collision>

File: armada_description/urdf/modules/mounts/mpm/mount.xacro (robot description, xacro)
@@ -16,4 +16,7 @@
                     <mesh filename="file://$(find armada_description)/meshes/modules/mounts/mpm/visual/mpm.stl" />
                 </geometry>
+                <material name="gray">
+                    <color rgba="0.7 0.7 0.7 1.0"/>
+                </material>
             </visual>
             <collision>

File: armada_description/urdf/modules/sensor_mounts/d435i_mount/sensor_mount.xacro (robot description, xacro)
@@ -16,4 +16,7 @@
                     <mesh filename="file://$(find armada_description)/meshes/modules/sensor_mounts/d435i_mount/visual/d435i_mount.stl" />
                 </geometry>
+                <material name="gray">
+                    <color rgba="0.7 0.7 0.7 1.0"/>
+                </material>
             </visual>
             <collision>
