Commit message: update name of stl file called by macro

File: armada_description/urdf/modules/tool_change_hardware/millibar/tool_changer.xacro (robot description, xacro)
@@ -14,10 +14,10 @@
             <visual>
                 <geometry>
-                    <mesh filename="file://$(find armada_description)/meshes/modules/tool_change_hardware/millibar/visual/millibar_adapters.stl" />
+                    <mesh filename="file://$(find armada_description)/meshes/modules/tool_change_hardware/millibar/visual/MTC-UR-Combined.stl" />
                 </geometry>
             </visual>
             <collision>
                 <geometry>
-                    <mesh filename="file://$(find armada_description)/meshes/modules/tool_change_hardware/millibar/collision/millibar_adapters.stl" />
+                    <mesh filename="file://$(find armada_description)/meshes/modules/tool_change_hardware/millibar/collision/MTC-UR-Combined.stl" />
                 </geometry>
             </collision>

Commit message: add material and color tag to visual geometry so model doesn't appear red; can be misinterpreted as a detected collision

File: armada_description/urdf/modules/tool_change_hardware/millibar/tool_changer.xacro (robot description, xacro)
@@ -16,4 +16,7 @@
                     <mesh filename="file://$(find armada_description)/meshes/modules/tool_change_hardware/millibar/visual/MTC-UR-Combined.stl" />
                 </geometry>
+                <material name="gray">
+                    <color rgba="0.7 0.7 0.7 1.0"/>
+                </material>
             </visual>
             <collision>
