Commit message: set default values for prefixes to blank, temporarily disable robotiq ros2 control macro call for debugging

File: armada_description/urdf/robot.urdf.xacro (robot description, xacro)
@@ -13,8 +13,10 @@
   <!-- Control Files -->
   <xacro:include filename="$(find armada_description)/urdf/modules/arms/$(arg model)/ros2_control.xacro"/>
-  <xacro:include filename="$(find armada_description)/urdf/modules/end_effectors/$(arg end_effector)/ros2_control.xacro"/>
+  <!-- <xacro:include filename="$(find armada_description)/urdf/modules/end_effectors/$(arg end_effector)/ros2_control.xacro"/> -->
   <!-- IMPORTANT: use tf_prefix, not prefix, and make it model-based -->
-  <xacro:arg name="arm_prefix" default="$(arg model)_"/>
-  <xacro:arg name="ee_prefix" default="$(arg end_effector)_"/>
+  <!-- <xacro:arg name="arm_prefix" default="$(arg model)_"/>
+  <xacro:arg name="ee_prefix" default="$(arg end_effector)_"/> -->
+  <xacro:arg name="arm_prefix" default=""/>
+  <xacro:arg name="ee_prefix" default=""/>
   <!-- Include your wrappers (not vendor macros directly) -->
   <xacro:include filename="$(find armada_description)/urdf/modules/arms/$(arg model)/arm.xacro"/>
@@ -28,7 +30,7 @@
   </xacro:armada_arm_ros2_control>
   <!-- Gripper ros2_control block -->
-  <xacro:armada_ee_ros2_control
+  <!-- <xacro:armada_ee_ros2_control
     prefix="" >
-  </xacro:armada_ee_ros2_control>
+  </xacro:armada_ee_ros2_control> -->
   <!-- World/root -->
   <link name="world"/>
@@ -36,5 +38,5 @@
   <xacro:armada_arm
     parent="world">
-    <origin xyz="0 0 1" rpy="0 0 0"/>
+    <origin xyz="0 0 0" rpy="0 0 0"/>
   </xacro:armada_arm>
   <!-- End-effector: attach directly to UR flange (sensor_mount removed) -->

Commit message: add in partially hard-coded armada_mount object for testing mount placement and functionality

File: armada_description/urdf/robot.urdf.xacro (robot description, xacro)
@@ -22,4 +22,6 @@
   <xacro:include filename="$(find armada_description)/urdf/modules/arms/$(arg model)/arm.xacro"/>
   <xacro:include filename="$(find armada_description)/urdf/modules/end_effectors/$(arg end_effector)/ee.xacro"/>
+  <!-- currently hard-code mount macro for testing -->
+  <xacro:include filename="$(find armada_description)/urdf/modules/mounts/mpm/mount.xacro"/>
   <!-- gazebo -->
   <!-- <xacro:arm_gazebo model="$(arg model)" /> -->
@@ -40,8 +42,16 @@
     <origin xyz="0 0 0" rpy="0 0 0"/>
   </xacro:armada_arm>
-  <!-- End-effector: attach directly to UR flange (sensor_mount removed) -->
+  <!-- parameterize mount prefix -->
+  <xacro:armada_mount
+    parent="$(arg arm_prefix)flange"
+    prefix="mpm_">
+    <!-- depth of socket center part is 6mm -->
+    <origin xyz="-0.006 0 0" rpy="0 0 0"/>
+  </xacro:armada_mount>
+  <!-- add logic, if mount then parent is mount, else arm flange -->
   <xacro:armada_ee
-    parent="$(arg arm_prefix)flange" >
-    <origin xyz="0 0 0" rpy="${pi/2} 0 ${pi/2}"/>
+    parent="mpm_base_link" >
+    <!-- 16mm along the x axis -->
+    <origin xyz="0.016 0 0" rpy="${pi/2} 0 ${pi/2}"/>
   </xacro:armada_ee>
 </robot>

Commit message: call armada_sensor_mount macro, test for functionality, deermine proper xyz placement

File: armada_description/urdf/robot.urdf.xacro (robot description, xacro)
@@ -24,4 +24,5 @@
   <!-- currently hard-code mount macro for testing -->
   <xacro:include filename="$(find armada_description)/urdf/modules/mounts/mpm/mount.xacro"/>
+  <xacro:include filename="$(find armada_description)/urdf/modules/sensor_mounts/d435i_mount/sensor_mount.xacro"/>
   <!-- gazebo -->
   <!-- <xacro:arm_gazebo model="$(arg model)" /> -->
@@ -50,4 +51,10 @@
     <origin xyz="-0.006 0 0" rpy="0 0 0"/>
   </xacro:armada_mount>
+  <xacro:armada_sensor_mount
+    parent="mpm_base_link"
+    prefix="d435i_mount_">
+    <!-- depth of sensor mount is 16mm, same thickness as mpm so no translation in x -->
+    <origin xyz="0 0 0.175" rpy="0 0 0"/>
+  </xacro:armada_sensor_mount>
   <!-- add logic, if mount then parent is mount, else arm flange -->
   <xacro:armada_ee

Commit message: update with macro for raspberry pi 5 controller

File: armada_description/urdf/robot.urdf.xacro (robot description, xacro)
@@ -25,4 +25,5 @@
   <xacro:include filename="$(find armada_description)/urdf/modules/mounts/mpm/mount.xacro"/>
   <xacro:include filename="$(find armada_description)/urdf/modules/sensor_mounts/d435i_mount/sensor_mount.xacro"/>
+  <xacro:include filename="$(find armada_description)/urdf/modules/controllers/rpi5_enclosure/controller.xacro"/>
   <!-- gazebo -->
   <!-- <xacro:arm_gazebo model="$(arg model)" /> -->
@@ -57,4 +58,10 @@
     <origin xyz="0 0 0.175" rpy="0 0 0"/>
   </xacro:armada_sensor_mount>
+  <xacro:armada_controller
+    parent="mpm_base_link"
+    prefix="rpi5_enclosure_">
+    <!-- depth of sensor mount is 16mm, same thickness as mpm so no translation in x -->
+    <origin xyz="-0.0325 0 0.175" rpy="0 0 0"/>
+  </xacro:armada_controller>
   <!-- add logic, if mount then parent is mount, else arm flange -->
   <xacro:armada_ee

Commit message: include and call macro to add realsense camera to robot, tweak origin values for positioning, calculate based on urdf values for camera

File: armada_description/urdf/robot.urdf.xacro (robot description, xacro)
@@ -3,4 +3,5 @@
   <!-- Generic-ish selectors -->
   <xacro:arg name="model" default="ur5e"/>
+  <xacro:arg name="sensor" default="d435i"/>
   <xacro:arg name="arm_ip" default="10.10.10.152"/>
   <xacro:arg name="end_effector" default="robotiq_2f85"/>
@@ -26,4 +27,5 @@
   <xacro:include filename="$(find armada_description)/urdf/modules/sensor_mounts/d435i_mount/sensor_mount.xacro"/>
   <xacro:include filename="$(find armada_description)/urdf/modules/controllers/rpi5_enclosure/controller.xacro"/>
+  <xacro:include filename="$(find armada_description)/urdf/modules/sensors/$(arg sensor)/sensor.xacro"/>
   <!-- gazebo -->
   <!-- <xacro:arm_gazebo model="$(arg model)" /> -->
@@ -64,4 +66,8 @@
     <origin xyz="-0.0325 0 0.175" rpy="0 0 0"/>
   </xacro:armada_controller>
+  <xacro:armada_sensor
+    parent="d435i_mount_base_link">
+    <origin xyz="0.024675 0 -0.0125" rpy="0 0 0"/>
+  </xacro:armada_sensor>
   <!-- add logic, if mount then parent is mount, else arm flange -->
   <xacro:armada_ee

Commit message: overhaul + refactor; pair wrappers with macros and build functional conditional blocks for modulatiry, add tool changer module, add block headers for more easy observation, remove hard coded name values values, TODO: remove hard coded origin values where possible; build them into the module xacro wrappers while still allowing offsets from modular robot.urdf.xacro macro

File: armada_description/urdf/robot.urdf.xacro (robot description, xacro)
@@ -1,78 +1,167 @@
 <?xml version="1.0"?>
 <robot name="armada_robot" xmlns:xacro="http://ros.org/wiki/xacro">
-  <!-- Generic-ish selectors -->
-  <xacro:arg name="model" default="ur5e"/>
-  <xacro:arg name="sensor" default="d435i"/>
-  <xacro:arg name="arm_ip" default="10.10.10.152"/>
-  <xacro:arg name="end_effector" default="robotiq_2f85"/>
-  <xacro:arg name="ee_ip" default="0.0.0.0"/>
-  <!-- ros2_control toggles (viewer should default off) -->
-  <xacro:arg name="use_ros2_control" default="false"/>
-  <xacro:arg name="sim_gazebo" default="false"/>
-  <!-- Gazebo plugin wrapper -->
+  <!-- ============================================================ -->
+  <!--                             ARGS                             -->
+  <!-- ============================================================ -->
+  <!-- Robot Environment -->
+  <xacro:arg name="root_link" default="world"/>
+  <!-- Robot Embodiment Selectors (explore armada_description/urdf/modules for options) -->
+  <xacro:arg name="arm" default=""/>
+  <xacro:arg name="mount" default=""/>
+  <xacro:arg name="sensor" default=""/>
+  <xacro:arg name="controller" default=""/>
+  <xacro:arg name="tool_change_hardware" default=""/>
+  <xacro:arg name="end_effector" default=""/>
+  <!-- Hardware IP Addresses -->
+  <xacro:arg name="arm_ip" default=""/>
+  <xacro:arg name="ee_ip" default=""/>
+  <!-- Simulation Toggle (should allow choosing simulator and be blank by default; TODO) -->
+  <xacro:arg name="simulator" default=""/>
+  <!-- Simulation plugin wrapper -->
   <!-- <xacro:include filename="$(find armada_gazebo)/xacro/modules/arms/$(arg model)/macro.gazebo.xacro"/> -->
-  <!-- Control Files -->
-  <xacro:include filename="$(find armada_description)/urdf/modules/arms/$(arg model)/ros2_control.xacro"/>
-  <!-- <xacro:include filename="$(find armada_description)/urdf/modules/end_effectors/$(arg end_effector)/ros2_control.xacro"/> -->
-  <!-- IMPORTANT: use tf_prefix, not prefix, and make it model-based -->
-  <!-- <xacro:arg name="arm_prefix" default="$(arg model)_"/>
-  <xacro:arg name="ee_prefix" default="$(arg end_effector)_"/> -->
-  <xacro:arg name="arm_prefix" default=""/>
-  <xacro:arg name="ee_prefix" default=""/>
-  <!-- Include your wrappers (not vendor macros directly) -->
-  <xacro:include filename="$(find armada_description)/urdf/modules/arms/$(arg model)/arm.xacro"/>
-  <xacro:include filename="$(find armada_description)/urdf/modules/end_effectors/$(arg end_effector)/ee.xacro"/>
-  <!-- currently hard-code mount macro for testing -->
-  <xacro:include filename="$(find armada_description)/urdf/modules/mounts/mpm/mount.xacro"/>
-  <xacro:include filename="$(find armada_description)/urdf/modules/sensor_mounts/d435i_mount/sensor_mount.xacro"/>
-  <xacro:include filename="$(find armada_description)/urdf/modules/controllers/rpi5_enclosure/controller.xacro"/>
-  <xacro:include filename="$(find armada_description)/urdf/modules/sensors/$(arg sensor)/sensor.xacro"/>
-  <!-- gazebo -->
-  <!-- <xacro:arm_gazebo model="$(arg model)" /> -->
-  <!-- Arm ros2_control block -->
-  <xacro:armada_arm_ros2_control
-    prefix="$(arg arm_prefix)"
-    robot_ip="$(arg arm_ip)"
-    model="$(arg model)" >
-  </xacro:armada_arm_ros2_control>
-  <!-- Gripper ros2_control block -->
-  <!-- <xacro:armada_ee_ros2_control
-    prefix="" >
-  </xacro:armada_ee_ros2_control> -->
-  <!-- World/root -->
-  <link name="world"/>
-  <!-- Arm: same scene placement you used before -->
+  <!-- ============================================================ -->
+  <!--                        ROS2 CONTROL                          -->
+  <!-- ============================================================ -->
+  <!-- Arm Physical Hardware Conditional Block -->
+  <xacro:if value="${'$(arg arm_ip)' != ''}">
+    <!-- Control File Wrapper -->
+    <xacro:include filename="$(find armada_description)/urdf/modules/arms/$(arg arm)/ros2_control.xacro"/>
+    <!-- Arm ros2_control block -->
+    <xacro:armada_arm_ros2_control
+      prefix="$(arg arm_prefix)"
+      robot_ip="$(arg arm_ip)"
+      model="$(arg arm)" >
+    </xacro:armada_arm_ros2_control>
+  </xacro:if>
+  <!-- End Effector Physical Hardware Conditional Block -->
+  <xacro:if value="${'$(arg ee_ip)' != '' and '$(arg end_effector)' != ''}">
+    <!-- Control File Wrapper -->
+    <xacro:include filename="$(find armada_description)/urdf/modules/end_effectors/$(arg end_effector)/ros2_control.xacro"/>
+    <!-- End Effector ros2_control block -->
+    <xacro:armada_ee_ros2_control
+      prefix="" >
+    </xacro:armada_ee_ros2_control>
+  </xacro:if>
+  <!-- ============================================================ -->
+  <!--                          ROOT LINK                           -->
+  <!-- ============================================================ -->
+  <!-- root link will be artificial "world" link unless alternate root link is passed to macro -->
+  <!-- World/Root Link Conditional Block -->
+  <xacro:if value="${'$(arg root_link)' == 'world'}">
+    <!-- World/Root Link-->
+    <link name="world"/>
+  </xacro:if>
+  <!-- ============================================================ -->
+  <!--                             ARM                              -->
+  <!-- ============================================================ -->
+  <!-- Arm Wrapper -->
+  <xacro:include filename="$(find armada_description)/urdf/modules/arms/$(arg arm)/arm.xacro"/>
+  <!-- Arm Macro -->
   <xacro:armada_arm
-    parent="world" >
+    parent="$(arg root_link)"
+    tf_prefix="$(arg arm)_" >
     <origin xyz="0 0 0" rpy="0 0 0"/>
   </xacro:armada_arm>
-  <!-- parameterize mount prefix -->
-  <xacro:armada_mount
-    parent="$(arg arm_prefix)flange"
-    prefix="mpm_">
-    <!-- depth of socket center part is 6mm -->
-    <origin xyz="-0.006 0 0" rpy="0 0 0"/>
-  </xacro:armada_mount>
-  <xacro:armada_sensor_mount
-    parent="mpm_base_link"
-    prefix="d435i_mount_">
-    <!-- depth of sensor mount is 16mm, same thickness as mpm so no translation in x -->
-    <origin xyz="0 0 0.175" rpy="0 0 0"/>
-  </xacro:armada_sensor_mount>
-  <xacro:armada_controller
-    parent="mpm_base_link"
-    prefix="rpi5_enclosure_">
-    <!-- depth of sensor mount is 16mm, same thickness as mpm so no translation in x -->
-    <origin xyz="-0.0325 0 0.175" rpy="0 0 0"/>
-  </xacro:armada_controller>
-  <xacro:armada_sensor
-    parent="d435i_mount_base_link">
-    <origin xyz="0.024675 0 -0.0125" rpy="0 0 0"/>
-  </xacro:armada_sensor>
-  <!-- add logic, if mount then parent is mount, else arm flange -->
-  <xacro:armada_ee
-    parent="mpm_base_link" >
-    <!-- 16mm along the x axis -->
-    <origin xyz="0.016 0 0" rpy="${pi/2} 0 ${pi/2}"/>
-  </xacro:armada_ee>
-</robot>
+  <!-- ============================================================ -->
+  <!--                       PERIPHERAL MOUNT                       -->
+  <!-- ============================================================ -->
+  <!-- (custom or additional hardware to interface between arm and peripherals) -->
+  <!-- Mount Conditional Block -->
+  <xacro:if value="${'$(arg mount)' != ''}">
+    <!-- Mount Wrapper -->
+    <xacro:include filename="$(find armada_description)/urdf/modules/mounts/$(arg mount)/mount.xacro"/>
+    <!-- Peripheral Mount Macro -->
+    <xacro:armada_mount
+      parent="$(arg arm)_flange"
+      prefix="$(arg mount)_">
+      <!-- depth of socket center part is 6mm -->
+      <origin xyz="-0.006 0 0" rpy="0 0 0"/>
+    </xacro:armada_mount>
+  </xacro:if>
+  <!-- ============================================================ -->
+  <!--                            SENSOR                            -->
+  <!-- ============================================================ -->
+  <!-- (e.g., depth sensors, cameras, lidar, etc.)-->
+  <!-- Sensor Conditional Block -->
+  <xacro:if value="${'$(arg sensor)' != ''}">
+    <!-- Sensor Wrappers -->
+    <xacro:include filename="$(find armada_description)/urdf/modules/sensors/$(arg sensor)/sensor.xacro"/>
+    <xacro:include filename="$(find armada_description)/urdf/modules/sensor_mounts/$(arg sensor)_mount/sensor_mount.xacro"/>
+    <!-- Sensor Mount Macro -->
+    <xacro:armada_sensor_mount
+      parent="$(arg mount)_base_link"
+      prefix="$(arg sensor)_mount_">
+      <!-- depth of sensor mount is 16mm, same thickness as mpm so no translation in x -->
+      <origin xyz="0 0 0.175" rpy="0 0 0"/>
+    </xacro:armada_sensor_mount>
+    <!-- Sensor Macro (e.g., camera, vision system, etc.)-->
+    <xacro:armada_sensor
+      parent="$(arg sensor)_mount_base_link">
+      <origin xyz="0.024675 0 -0.0125" rpy="0 0 0"/>
+    </xacro:armada_sensor>
+  </xacro:if>
+  <!-- ============================================================ -->
+  <!--                          CONTROLLER                          -->
+  <!-- ============================================================ -->
+  <!-- (e.g., raspberry pi 5 for sensor and gripper control + networking) -->
+  <!-- Controller Conditional Block -->
+  <xacro:if value="${'$(arg controller)' != ''}">
+    <!-- Controller Wrapper -->
+    <xacro:include filename="$(find armada_description)/urdf/modules/controllers/$(arg controller)_enclosure/controller.xacro"/>
+    <!-- Controller Macro -->
+    <xacro:armada_controller
+      parent="$(arg mount)_base_link"
+      prefix="$(arg controller)_enclosure_">
+      <!-- depth of sensor mount is 16mm, same thickness as mpm so no translation in x -->
+      <origin xyz="-0.0325 0 0.175" rpy="0 0 0"/>
+    </xacro:armada_controller>
+  </xacro:if>
+  <!-- ============================================================ -->
+  <!--                      TOOL CHANGE HARDWARE                    -->
+  <!-- ============================================================ -->
+  <!-- (e.g., millibar or some other 3rd party or custom tool change hardware for robot tooling) -->
+  <!-- Quick Change Hardware Conditional Block -->
+  <xacro:if value="${'$(arg tool_change_hardware)' != ''}">
+    <!-- Conditional Robot Embodiment Selector -->
+    <xacro:property
+      name="tool_changer_parent"
+      value="${'$(arg arm)' + '_flange' if '$(arg mount)' == '' else '$(arg mount)' + '_base_link'}">
+    </xacro:property>
+    <!-- Quick Change Hardware Wrapper -->
+    <xacro:include filename="$(find armada_description)/urdf/modules/tool_change_hardware/$(arg tool_change_hardware)/tool_changer.xacro"/>
+    <!-- Quick Change Hardware Macro -->
+    <xacro:armada_tool_changer
+      parent="${tool_changer_parent}"
+      prefix="$(arg tool_change_hardware)_" >
+      <!-- 16mm along the x axis -->
+      <origin xyz="0.016 0 0" rpy="0 0 0"/>
+    </xacro:armada_tool_changer>
+  </xacro:if>
+  <!-- ============================================================ -->
+  <!--                         END EFFECTOR                         -->
+  <!-- ============================================================ -->
+  <!-- Conditional Robot Embodiment Selector -->
+  <xacro:property
+    name="ee_parent"
+    value="${
+      '$(arg tool_change_hardware)' + '_base_link'
+        if '$(arg tool_change_hardware)' != ''
+      else
+      '$(arg mount)' + '_base_link'
+        if '$(arg mount)' != ''
+      else
+      '$(arg arm)' + '_flange'
+    }">
+  </xacro:property>
+  <!-- End Effector Conditional Block -->
+  <xacro:if value="${'$(arg end_effector)' != ''}">
+    <!-- End Effector Wrapper -->
+    <xacro:include filename="$(find armada_description)/urdf/modules/end_effectors/$(arg end_effector)/ee.xacro"/>
+    <!-- End Effector Macro -->
+    <xacro:armada_ee
+      parent="${ee_parent}" >
+      <!-- 16mm along the x axis -->
+      <origin xyz="0.016 0 0" rpy="${pi/2} 0 ${pi/2}"/>
+    </xacro:armada_ee>
+  </xacro:if>
+</robot> <!-- armada_robot -->

Commit message: update origin of end effector with respect to millibar adapters, TODO; still hard-coded, need a way to programatically add this value

File: armada_description/urdf/robot.urdf.xacro (robot description, xacro)
@@ -162,5 +162,5 @@
       parent="${ee_parent}" >
       <!-- 16mm along the x axis -->
-      <origin xyz="0.016 0 0" rpy="${pi/2} 0 ${pi/2}"/>
+      <origin xyz="0.03244 0 0" rpy="${pi/2} 0 ${pi/2}"/>
     </xacro:armada_ee>
   </xacro:if>

Commit message: find better value for realsense camera offset (sensor origin with respect to sensor mount plate)

File: armada_description/urdf/robot.urdf.xacro (robot description, xacro)
@@ -98,5 +98,5 @@
     <xacro:armada_sensor
       parent="$(arg sensor)_mount_base_link">
-      <origin xyz="0.024675 0 -0.0125" rpy="0 0 0"/>
+      <origin xyz="0.0260125 0 -0.0125" rpy="0 0 0"/>
     </xacro:armada_sensor>
   </xacro:if>

Commit message: adjust gripper offset distance, remove unnecessary or inaccurate comments from macro blocks, add simulation macro block for future

File: armada_description/urdf/robot.urdf.xacro (robot description, xacro)
@@ -18,4 +18,7 @@
   <!-- Simulation Toggle (should allow choosing simulator and be blank by default; TODO) -->
   <xacro:arg name="simulator" default=""/>
+  <!-- ============================================================ -->
+  <!--                         SIMULATION                           -->
+  <!-- ============================================================ -->
   <!-- Simulation plugin wrapper -->
   <!-- <xacro:include filename="$(find armada_gazebo)/xacro/modules/arms/$(arg model)/macro.gazebo.xacro"/> -->
@@ -75,5 +78,4 @@
       parent="$(arg arm)_flange"
       prefix="$(arg mount)_">
-      <!-- depth of socket center part is 6mm -->
       <origin xyz="-0.006 0 0" rpy="0 0 0"/>
     </xacro:armada_mount>
@@ -92,5 +94,4 @@
       parent="$(arg mount)_base_link"
       prefix="$(arg sensor)_mount_">
-      <!-- depth of sensor mount is 16mm, same thickness as mpm so no translation in x -->
       <origin xyz="0 0 0.175" rpy="0 0 0"/>
     </xacro:armada_sensor_mount>
@@ -113,5 +114,4 @@
       parent="$(arg mount)_base_link"
       prefix="$(arg controller)_enclosure_">
-      <!-- depth of sensor mount is 16mm, same thickness as mpm so no translation in x -->
       <origin xyz="-0.0325 0 0.175" rpy="0 0 0"/>
     </xacro:armada_controller>
@@ -134,5 +134,4 @@
       parent="${tool_changer_parent}"
       prefix="$(arg tool_change_hardware)_" >
-      <!-- 16mm along the x axis -->
       <origin xyz="0.016 0 0" rpy="0 0 0"/>
     </xacro:armada_tool_changer>
@@ -161,6 +160,6 @@
     <xacro:armada_ee
       parent="${ee_parent}" >
-      <!-- 16mm along the x axis -->
-      <origin xyz="0.03244 0 0" rpy="${pi/2} 0 ${pi/2}"/>
+      <!-- 0.03244 -->
+      <origin xyz="0.03394 0 0" rpy="${pi/2} 0 ${pi/2}"/>
     </xacro:armada_ee>
   </xacro:if>

Commit message: rotate peripheral mount by 180 degrees around x axis (roll)

File: armada_description/urdf/robot.urdf.xacro (robot description, xacro)
@@ -78,5 +78,5 @@
       parent="$(arg arm)_flange"
       prefix="$(arg mount)_">
-      <origin xyz="-0.006 0 0" rpy="0 0 0"/>
+      <origin xyz="-0.006 0 0" rpy="3.14 0 0"/>
     </xacro:armada_mount>
   </xacro:if>
